File: Controller/ECEN1400_Board/schematic.sch (EAGLE design)
At the start: 49 parts, among them Q1 500mA/300V, Q2 500mA/300V, Q3 500mA/300V, Q4 500mA/300V, Q5 500mA/300V, Q6 500mA/300V, U1 MCP73831, U2 MCP73831, U3 3.3V, U4 LM1117, U5 ATSAMD21G-A, Y1 32.768kHz

Commit message: Added L293D class and beginning of custom weather board
Parts:
- removed C7: 1.0uF, SparkFun-Capacitors:1.0UF-1206-50V-10%
- removed C8: 2.2uF, SparkFun-Capacitors:2.2UF-1206-50V-10%
- removed D3, D4: (no value), SparkFun-LED:LED-FKIT-1206
- removed J2: (no value), SparkFun-Connectors:M021X02_NO_SILK
- removed Q1, Q2, Q3, Q4, Q5, Q6: 500mA/300V, SparkFun-DiscreteSemi:TRANS_NPN-MMBTA42
- removed R7: 470, SparkFun-Resistors:0.1OHM-1210-1/2W-1%
- removed U4: LM1117, LM1117_2:LM1117
- added F1: 6V/0.5A, SparkFun-Fuses:PPTC_HALF-AMP
- C10, C11, C9: value 0.1uF -> 1.0uF
- C3: value 4.7uF -> 1.0uF; device SparkFun-Capacitors:10UF-1206-6.3V-20% -> SparkFun-Capacitors:1.0UF-1206-50V-10%
- C4: value 10uF -> 1.0uF; device SparkFun-Capacitors:10UF-1206-6.3V-20% -> SparkFun-Capacitors:1.0UF-1206-50V-10%
- C6: value 2.2uF -> 1.0uF; device SparkFun-Capacitors:2.2UF-1206-50V-10% -> SparkFun-Capacitors:1.0UF-1206-50V-10%
- R1: value 700 -> 470
- R3: value 4K -> 2K
- R4: value 470 -> 4.7K
- R5: value 4K -> 180
- R6: value 470 -> 1K
- U$1: value (none) -> SWITCH_SPDT; device custom:JS207011SCQNR -> SparkFun-Retired:SWITCH_SPDT
- U2: value MCP73831 -> 3.3V; device SparkFun-IC-Power:MCP73831 -> SparkFun-IC-Power:V_REG_AP2112K-3.3V
- U3: value 3.3V -> MAX1704X; device SparkFun-IC-Power:V_REG_AP2112K-3.3V -> SparkFun-IC-Power:MAX1704X
Connections:
- removed net 12V: C1.1, C10.1, C11.1, C3.1, C6.1, C8.1, D3.A, D4.A, J2.2, J6.2, Q5.E, Q6.E, R9.2, S1.VCC, U1.VBAT, U2.VBAT, U3.OUT, U4.VO, U5.VDDANA, U5.VDDIN, U5.VDDIO@17, U5.VDDIO@36
- removed net A0/2: S1.X
- removed net A1/2: S1.Y
- removed net CHG_SW: Q1.B, Q2.B, Q3.B, U$1.6
- removed net D2/2: S2.2
- removed net D3/2: S3.2
- removed net D4/2: S4.2
- removed net D5/2: S5.2
- removed net GND1: C12.1, C13.1
- removed net N$10: J2.1, Q3.E, Q4.E
- removed net N$11: C5.1, Q5.C, U3.EN, U3.IN
- removed net N$12: C7.1, Q6.C, U4.VI
- removed net N$13: D3.C, R7.2
- removed net N$14: D4.C, R6.2
- removed net N$9: R5.2, U2.PROG
- removed net OFF_SW: U$1.5
- removed net ON_SW: Q4.B, Q5.B, Q6.B, U$1.8
- removed net V_3.7: Q4.C
- removed net V_USB: Q1.E, Q2.E
- new net 3.3V: C10.1, C11.1, C3.1, D2.A, R4.2, R6.2, R9.2, S1.VCC, U$1.S, U2.OUT, U5.VDDANA, U5.VDDIN, U5.VDDIO@17, U5.VDDIO@36
- new net SCL/2: U3.SCL
- new net SDA/2: U3.SDA
- new net USB_HOST_EN/1: J1.ID
- new net VIN: C2.1, C4.1, F1.2, R2.2, U1.VIN, U2.IN
- new net V_BATT: C1.1, J6.2, R5.2, U1.VBAT
- net A0/1: now also S1.X
- net A1/1: now also S1.Y
- net D2/1: now also S2.2
- net D3/1: now also S3.2
- net D4/1: now also S4.2
- net D5/1: now also S5.2
- net D7/1: now also R4.1, U3.ALT
- net GND: now also C12.1, C13.1, J1.GND, R1.1, U$1.O, U2.GND, U3.CTG, U3.GND@4, U3.GND@EP, U3.QST; no longer C7.2, C8.2, Q3.C, R1.2, R5.1, R6.1, R7.1, U2.VSS, U3.GND, U4.GND
- net N$1: now also C5.1, R6.1, U3.VDD; no longer R1.1, U$1.7
- net N$15: now also U5.PA00(XIN32/SER1:0/TC2:0)
- net N$2: now also C6.1, R5.1, U3.CELL; no longer C2.1, Q1.C, R2.2, U1.VIN
- net N$22: now also U5.PA01(XOUT32/SER1:1/TC2:1)
- net N$5: now also U$1.P, U2.EN; no longer C4.1, Q2.C, R4.2, U2.VIN
- net N$7: now also F1.1, J1.VBUS; no longer D2.A, R4.1
- net N$8: now also R1.2; no longer U2.STAT
- net USB_D+/1: now also J1.D+
- net USB_D-/1: now also J1.D-
Other:
- moved on the sheet: C3, C4, C5, C6, D2, J1, R1, R4, R5, R6
